File: spindle_controller.sch (KiCad schematic (older format))
At the start: 57 parts, among them J1 VAC 230V, J2 AUX/CONTROL, J3 ICP, J4 Load output, J5 CONN_01X03, J6 CONN_01X03, Q1 2N3904, SW1 Rotary_Encoder_Switch, T1 230 - 6VAC (Spitznagel SPK 01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, U1 7805, U2 ATMEGA328P-PU, U3 PC817, U4 MOC3020M, U5 TCRT5000, Y1 16MHz

Commit message: Add board routing halfway
Parts:
- removed U1: 7805, Power_Integrations:TO-220, symbol 7805
- added CASE?: Case, iotta_footprints:CASE_KEMO_G085N, symbol iotta_logo
- added U1: LM7805CT, TO_SOT_Packages_THT:TO-220_Vertical, symbol LM7805CT
- C16, C17: footprint Capacitors_ThroughHole:C_Rect_L7.0mm_W2.5mm_P5.00mm -> Capacitors_ThroughHole:C_Rect_L16.5mm_W5.0mm_P15.00mm_MKT
- D7: footprint Power_Integrations:TO-220 -> TO_SOT_Packages_THT:TO-220_Vertical
- R16: footprint Resistors_ThroughHole:R_Axial_DIN0204_L3.6mm_D1.6mm_P7.62mm_Horizontal -> Resistors_ThroughHole:R_Axial_DIN0414_L11.9mm_D4.5mm_P15.24mm_Horizontal
- T1: symbol Transformer_1P_1S -> Transformer_spitznagel_SPK01406
Connections:
- net GND: now also U1.2 (GND)
- net VCC: now also U1.3 (OUT)
- net VAC_L: now reaches C16.1, D7.2 (A1), J1.2, R6.2, R8.2, T1.1 (AA)
- net VAC_N: now reaches J1.1, J4.1, R3.2
- net VAC_N: now also T1.5 (AB); no longer T1.2 (AB)
- net at C11.1, D2.2 (A), R4.1: now also D3.1 (K); no longer D3.2 (A)
- net at C11.2, D6.1 (K), R7.1: now also D4.2 (A); no longer D4.1 (K)
- net at C10.1, D2.1 (K), R2.2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: now also D4.1 (K); no longer D3.1 (K)
- net at D5.1 (K), D6.2 (A), Q1.2 (B)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: now also D3.2 (A); no longer D4.2 (A)
- net at C3.1, C4.1, D1.1 (+): now also U1.1 (IN)
- net at D1.2: now also T1.9 (SA); no longer T1.3 (SA)
- net at D1.3: now also T1.7 (SB); no longer T1.4 (SB)
Other:
- moved on the sheet: J4, R5
Changed lines of the file:
@@
 F 0 "D7" H 2828 5296 50  0000 L CNN
 F 1 "BT138" H 2828 5205 50  0000 L CNN
-F 2 "Power_Integrations:TO-220" V 2775 5275 50  0001 C CNN
+F 2 "TO_SOT_Packages_THT:TO-220_Vertical" V 2775 5275 50  0001 C CNN
 F 3 "" V 2700 5250 50  0001 C CNN
 	1    2700 5250
@@
 F 3 "" H 3050 3300 50  0001 C CNN
 	1    3050 3300
-	-1   0    0    1
+	1    0    0    -1
 $EndComp
 $Comp
@@
 F 3 "" H 3050 3700 50  0001 C CNN
 	1    3050 3700
-	1    0    0    -1
+	-1   0    0    1
 $EndComp
 $Comp
@@
 L R R5
 U 1 1 58F0B508
-P 3400 3500
-F 0 "R5" H 3330 3454 50  0000 R CNN
-F 1 "33k" H 3330 3545 50  0000 R CNN
-F 2 "Resistors_ThroughHole:R_Axial_DIN0204_L3.6mm_D1.6mm_P7.62mm_Horizontal" V 3330 3500 50  0001 C CNN
-F 3 "" H 3400 3500 50  0001 C CNN
-	1    3400 3500
+P 3850 3500
+F 0 "R5" H 3780 3454 50  0000 R CNN
+F 1 "33k" H 3780 3545 50  0000 R CNN
+F 2 "Resistors_ThroughHole:R_Axial_DIN0204_L3.6mm_D1.6mm_P7.62mm_Horizontal" V 3780 3500 50  0001 C CNN
+F 3 "" H 3850 3500 50  0001 C CNN
+	1    3850 3500
 	-1   0    0    1
 $EndComp
@@
 $EndComp
 $Comp
-L GND #PWR6
+L GND #PWR01
 U 1 1 58F0C844
 P 5900 3450
-F 0 "#PWR6" H 5900 3200 50  0001 C CNN
+F 0 "#PWR01" H 5900 3200 50  0001 C CNN
 F 1 "GND" H 5905 3277 50  0000 C CNN
 F 2 "" H 5900 3450 50  0001 C CNN
@@
 $EndComp
 $Comp
-L VCC #PWR5
+L VCC #PWR02
 U 1 1 58F0CA70
 P 5900 2650
-F 0 "#PWR5" H 5900 2500 50  0001 C CNN
+F 0 "#PWR02" H 5900 2500 50  0001 C CNN
 F 1 "VCC" H 5917 2823 50  0000 C CNN
 F 2 "" H 5900 2650 50  0001 C CNN
@@
 L Screw_Terminal_1x02 J4
 U 1 1 58F0D457
-P 950 5400
-F 0 "J4" H 1030 5742 50  0000 C CNN
-F 1 "Load output" H 1030 5651 50  0000 C CNN
-F 2 "Terminal_Blocks:TerminalBlock_Pheonix_MKDS1.5-2pol" H 950 5175 50  0001 C CNN
-F 3 "" H 925 5400 50  0001 C CNN
-	1    950  5400
+P 750 5400
+F 0 "J4" H 830 5742 50  0000 C CNN
+F 1 "Load output" H 830 5651 50  0000 C CNN
+F 2 "Terminal_Blocks:TerminalBlock_Pheonix_MKDS1.5-2pol" H 750 5175 50  0001 C CNN
+F 3 "" H 725 5400 50  0001 C CNN
+	1    750  5400
 	1    0    0    -1
 $EndComp
@@
 F 0 "C17" H 3515 5196 50  0000 L CNN
 F 1 "1n" H 3515 5105 50  0000 L CNN
-F 2 "Capacitors_ThroughHole:C_Rect_L7.0mm_W2.5mm_P5.00mm" H 3438 5000 50  0001 C CNN
+F 2 "Capacitors_ThroughHole:C_Rect_L16.5mm_W5.0mm_P15.00mm_MKT" H 3438 5000 50  0001 C CNN
 F 3 "" H 3400 5150 50  0001 C CNN
 	1    3400 5150
@@
 F 0 "C16" H 2315 5096 50  0000 L CNN
 F 1 "10n" H 2315 5005 50  0000 L CNN
-F 2 "Capacitors_ThroughHole:C_Rect_L7.0mm_W2.5mm_P5.00mm" H 2238 4900 50  0001 C CNN
+F 2 "Capacitors_ThroughHole:C_Rect_L16.5mm_W5.0mm_P15.00mm_MKT" H 2238 4900 50  0001 C CNN
 F 3 "" H 2200 5050 50  0001 C CNN
 	1    2200 5050
@@
 F 0 "R16" H 2130 5404 50  0000 R CNN
 F 1 "47" H 2130 5495 50  0000 R CNN
-F 2 "Resistors_ThroughHole:R_Axial_DIN0204_L3.6mm_D1.6mm_P7.62mm_Horizontal" V 2130 5450 50  0001 C CNN
+F 2 "Resistors_ThroughHole:R_Axial_DIN0414_L11.9mm_D4.5mm_P15.24mm_Horizontal" V 2130 5450 50  0001 C CNN
 F 3 "" H 2200 5450 50  0001 C CNN
 	1    2200 5450
@@
 $EndComp
 $Comp
-L GND #PWR16
+L GND #PWR03
 U 1 1 58F0F278
 P 4750 5100
-F 0 "#PWR16" H 4750 4850 50  0001 C CNN
+F 0 "#PWR03" H 4750 4850 50  0001 C CNN
 F 1 "GND" H 4755 4927 50  0000 C CNN
 F 2 "" H 4750 5100 50  0001 C CNN
@@
 $EndComp
 $Comp
-L GND #PWR7
+L GND #PWR04
 U 1 1 58F119B3
 P 10300 3600
-F 0 "#PWR7" H 10300 3350 50  0001 C CNN
+F 0 "#PWR04" H 10300 3350 50  0001 C CNN
 F 1 "GND" H 10305 3427 50  0000 C CNN
 F 2 "" H 10300 3600 50  0001 C CNN
@@
 $EndComp
 $Comp
-L VCC #PWR2
+L VCC #PWR05
 U 1 1 58F11EE3
 P 10300 950
-F 0 "#PWR2" H 10300 800 50  0001 C CNN
+F 0 "#PWR05" H 10300 800 50  0001 C CNN
 F 1 "VCC" H 10317 1123 50  0000 C CNN
 F 2 "" H 10300 950 50  0001 C CNN
 F 3 "" H 10300 950 50  0001 C CNN
 	1    10300 950
-	1    0    0    -1
-$EndComp
-$Comp
-L 7805 U1
-U 1 1 58F122A6
-P 4800 1100
-F 0 "U1" H 4800 1415 50  0000 C CNN
-F 1 "7805" H 4800 1324 50  0000 C CNN
-F 2 "Power_Integrations:TO-220" H 4800 1100 50  0001 C CNN
-F 3 "" H 4800 1100 50  0001 C CNN
-	1    4800 1100
 	1    0    0    -1
 $EndComp
@@
 $EndComp
 $Comp
-L VCC #PWR1
+L VCC #PWR06
 U 1 1 58F13E70
 P 5900 950
-F 0 "#PWR1" H 5900 800 50  0001 C CNN
+F 0 "#PWR06" H 5900 800 50  0001 C CNN
 F 1 "VCC" H 5917 1123 50  0000 C CNN
 F 2 "" H 5900 950 50  0001 C CNN
@@
 $EndComp
 $Comp
-L GND #PWR3
+L GND #PWR07
 U 1 1 58F13F62
 P 5900 1950
-F 0 "#PWR3" H 5900 1700 50  0001 C CNN
+F 0 "#PWR07" H 5900 1700 50  0001 C CNN
 F 1 "GND" H 5905 1777 50  0000 C CNN
 F 2 "" H 5900 1950 50  0001 C CNN
@@
 $EndComp
 $Comp
-L GND #PWR17
+L GND #PWR08
 U 1 1 58F18A24
 P 7800 5650
-F 0 "#PWR17" H 7800 5400 50  0001 C CNN
+F 0 "#PWR08" H 7800 5400 50  0001 C CNN
 F 1 "GND" H 7805 5477 50  0000 C CNN
 F 2 "" H 7800 5650 50  0001 C CNN
@@
 ROT_PULSE
 $Comp
-L VCC #PWR13
+L VCC #PWR09
 U 1 1 58F19F6D
 P 7800 4750
-F 0 "#PWR13" H 7800 4600 50  0001 C CNN
+F 0 "#PWR09" H 7800 4600 50  0001 C CNN
 F 1 "VCC" H 7817 4923 50  0000 C CNN
 F 2 "" H 7800 4750 50  0001 C CNN
@@
 $EndComp
 $Comp
-L GND #PWR18
+L GND #PWR010
 U 1 1 58F1A44D
 P 10050 5950
-F 0 "#PWR18" H 10050 5700 50  0001 C CNN
+F 0 "#PWR010" H 10050 5700 50  0001 C CNN
 F 1 "GND" H 10055 5777 50  0000 C CNN
 F 2 "" H 10050 5950 50  0001 C CNN
@@
 $EndComp
 $Comp
-L VCC #PWR12
+L VCC #PWR011
 U 1 1 58F1BEE5
 P 10050 4700
-F 0 "#PWR12" H 10050 4550 50  0001 C CNN
+F 0 "#PWR011" H 10050 4550 50  0001 C CNN
 F 1 "VCC" H 10067 4873 50  0000 C CNN
 F 2 "" H 10050 4700 50  0001 C CNN
@@
 $EndComp
 $Comp
-L GND #PWR15
+L GND #PWR012
 U 1 1 58F1C6A9
 P 10850 5000
-F 0 "#PWR15" H 10850 4750 50  0001 C CNN
+F 0 "#PWR012" H 10850 4750 50  0001 C CNN
 F 1 "GND" H 10855 4827 50  0000 C CNN
 F 2 "" H 10850 5000 50  0001 C CNN
@@
 $EndComp
 $Comp
-L GND #PWR14
+L GND #PWR013
 U 1 1 58F1C89A
 P 7300 4950
-F 0 "#PWR14" H 7300 4700 50  0001 C CNN
+F 0 "#PWR013" H 7300 4700 50  0001 C CNN
 F 1 "GND" H 7305 4777 50  0000 C CNN
 F 2 "" H 7300 4950 50  0001 C CNN
@@
 SCK
 $Comp
-L GND #PWR19
+L GND #PWR014
 U 1 1 58F1DDC1
 P 1150 7500
-F 0 "#PWR19" H 1150 7250 50  0001 C CNN
+F 0 "#PWR014" H 1150 7250 50  0001 C CNN
 F 1 "GND" H 1155 7327 50  0000 C CNN
 F 2 "" H 1150 7500 50  0001 C CNN
@@
 $EndComp
 $Comp
-L GND #PWR11
+L GND #PWR015
 U 1 1 58F281AB
 P 9700 4350
-F 0 "#PWR11" H 9700 4100 50  0001 C CNN
+F 0 "#PWR015" H 9700 4100 50  0001 C CNN
 F 1 "GND" H 9705 4177 50  0000 C CNN
 F 2 "" H 9700 4350 50  0001 C CNN
@@
 $EndComp
 $Comp
-L GND #PWR10
+L GND #PWR016
 U 1 1 58F28222
 P 6600 4300
-F 0 "#PWR10" H 6600 4050 50  0001 C CNN
+F 0 "#PWR016" H 6600 4050 50  0001 C CNN
 F 1 "GND" H 6605 4127 50  0000 C CNN
 F 2 "" H 6600 4300 50  0001 C CNN
@@
 $EndComp
 $Comp
-L VCC #PWR8
+L VCC #PWR017
 U 1 1 58F28299
 P 6600 4000
-F 0 "#PWR8" H 6600 3850 50  0001 C CNN
+F 0 "#PWR017" H 6600 3850 50  0001 C CNN
 F 1 "VCC" H 6617 4173 50  0000 C CNN
 F 2 "" H 6600 4000 50  0001 C CNN
@@
 $EndComp
 $Comp
-L VCC #PWR9
+L VCC #PWR018
 U 1 1 58F28310
 P 9700 4050
-F 0 "#PWR9" H 9700 3900 50  0001 C CNN
+F 0 "#PWR018" H 9700 3900 50  0001 C CNN
 F 1 "VCC" H 9717 4223 50  0000 C CNN
 F 2 "" H 9700 4050 50  0001 C CNN
@@
 $EndComp
 $Comp
-L GND #PWR4
+L GND #PWR019
 U 1 1 58F2C665
 P 6600 2150
-F 0 "#PWR4" H 6600 1900 50  0001 C CNN
+F 0 "#PWR019" H 6600 1900 50  0001 C CNN
 F 1 "GND" H 6605 1977 50  0000 C CNN
 F 2 "" H 6600 2150 50  0001 C CNN
@@
 NoConn ~ 4350 250
 $Comp
-L Transformer_1P_1S T1
+L Transformer_spitznagel_SPK01406 T1
 U 1 1 58F121ED
 P 1900 1450
@@
 	3200 3000 4500 3000
 Wire Wire Line
-	3400 3000 3400 3350
-Wire Wire Line
-	3400 3300 3200 3300
-Connection ~ 3400 3300
-Wire Wire Line
-	3200 3700 3400 3700
-Wire Wire Line
-	3400 3650 3400 4000
+	3200 3300 3550 3300
 Wire Wire Line
 	3200 4000 4700 4000
-Connection ~ 3400 3700
 Wire Wire Line
 	4700 4000 4700 3850
-Connection ~ 3400 4000
 Wire Wire Line
 	4200 3950 4200 4000
@@
 Wire Wire Line
 	4200 3000 4200 3100
-Connection ~ 3400 3000
 Connection ~ 4200 3000
 Wire Wire Line
@@
 	1250 1250 1250 5300
 Wire Wire Line
-	1250 5300 1150 5300
+	1250 5300 950  5300
 Wire Wire Line
 	1450 4800 2950 4800
@@
 Connection ~ 2700 4800
 Wire Wire Line
-	1150 5500 1250 5500
+	950  5500 1250 5500
 Wire Wire Line
 	1250 5500 1250 5700
@@
 	4350 4350 4350 6050
 Wire Notes Line
-	4350 6050 750  6050
+	4350 6050 650  6050
 Wire Notes Line
 	1900 800  650  800
@@
 	1    0    0    -1
 $EndComp
+$Comp
+L LM7805CT U1
+U 1 1 58F0F97F
+P 4800 1100
+F 0 "U1" H 4800 1417 50  0000 C CNN
+F 1 "LM7805CT" H 4800 1326 50  0000 C CNN
+F 2 "TO_SOT_Packages_THT:TO-220_Vertical" H 4800 1200 50  0001 C CIN
+F 3 "" H 4800 1100 50  0001 C CNN
+	1    4800 1100
+	1    0    0    -1
+$EndComp
+Text Label 1250 3300 2    60   ~ 0
+VAC_N
+Text Label 1450 3700 2    60   ~ 0
+VAC_L
+Wire Wire Line
+	3550 3300 3550 4000
+Connection ~ 3550 4000
+Wire Wire Line
+	3200 3700 3400 3700
+Wire Wire Line
+	3400 3700 3400 3000
+Connection ~ 3400 3000
+Wire Wire Line
+	3850 3350 3850 3000
+Connection ~ 3850 3000
+Wire Wire Line
+	3850 3650 3850 4000
+Connection ~ 3850 4000
+$Comp
+L iotta_logo CASE?
+U 1 1 58F16C0B
+P 7150 6950
+F 0 "CASE?" H 7778 7103 60  0000 L CNN
+F 1 "Case" H 7778 7050 60  0001 L CNN
+F 2 "iotta_footprints:CASE_KEMO_G085N" H 7778 6997 60  0000 L CNN
+F 3 "" H 7150 6950 60  0000 C CNN
+	1    7150 6950
+	1    0    0    -1
+$EndComp

Commit message: Add shuffled AC cord entry, ziplock holes, 1117 regulator alternative, shuffled linear supply
Parts:
- added U6: AP111750, TO_SOT_Packages_SMD:SOT-223, symbol AP111750
- added WIRESTRAP1: 2x Ziplock wire strap, iotta_footprints:WireStrap_2X, symbol iotta_logo
- C17: footprint Capacitors_ThroughHole:C_Rect_L16.5mm_W5.0mm_P15.00mm_MKT -> Capacitors_ThroughHole:C_Disc_D8.0mm_W5.0mm_P7.50mm
- U1: footprint TO_SOT_Packages_THT:TO-220_Vertical -> TO_SOT_Packages_THT:TO-220_Horizontal
- gave numbers to parts that had none: 1
Connections:
- net GND: now also U6.1 (GND/ADJ)
- net VCC: now also U6.2 (VO), U6.4 (VO)
- net at C3.1, C4.1, D1.1 (+)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: now also U6.3 (VI)
- no-connect marks 10 -> 8
Other:
- note added: "1117 Regulator SMD alternative\nfor 7805 (place only one!)"
- moved on the sheet: C7, C9, Y1
Changed lines of the file:
@@
 F 0 "C17" H 3515 5196 50  0000 L CNN
 F 1 "1n" H 3515 5105 50  0000 L CNN
-F 2 "Capacitors_ThroughHole:C_Rect_L16.5mm_W5.0mm_P15.00mm_MKT" H 3438 5000 50  0001 C CNN
+F 2 "Capacitors_ThroughHole:C_Disc_D8.0mm_W5.0mm_P7.50mm" H 3438 5000 50  0001 C CNN
 F 3 "" H 3400 5150 50  0001 C CNN
 	1    3400 5150
@@
 L Crystal Y1
 U 1 1 58F2C410
-P 7100 1750
-F 0 "Y1" V 7054 1881 50  0000 L CNN
-F 1 "16MHz" V 7145 1881 50  0000 L CNN
-F 2 "Crystals:Crystal_HC49-U_Vertical" H 7100 1750 50  0001 C CNN
-F 3 "" H 7100 1750 50  0001 C CNN
-	1    7100 1750
+P 7350 1950
+F 0 "Y1" V 7304 2081 50  0000 L CNN
+F 1 "16MHz" V 7395 2081 50  0000 L CNN
+F 2 "Crystals:Crystal_HC49-U_Vertical" H 7350 1950 50  0001 C CNN
+F 3 "" H 7350 1950 50  0001 C CNN
+	1    7350 1950
 	0    1    1    0
 $EndComp
@@
 L C C7
 U 1 1 58F2C4B6
-P 6850 1500
-F 0 "C7" V 6598 1500 50  0000 C CNN
-F 1 "33p" V 6689 1500 50  0000 C CNN
-F 2 "Capacitors_ThroughHole:C_Rect_L4.6mm_W2.0mm_P2.50mm_MKS02_FKP02" H 6888 1350 50  0001 C CNN
-F 3 "" H 6850 1500 50  0001 C CNN
-	1    6850 1500
+P 7100 1700
+F 0 "C7" V 6848 1700 50  0000 C CNN
+F 1 "33p" V 6939 1700 50  0000 C CNN
+F 2 "Capacitors_ThroughHole:C_Rect_L4.6mm_W2.0mm_P2.50mm_MKS02_FKP02" H 7138 1550 50  0001 C CNN
+F 3 "" H 7100 1700 50  0001 C CNN
+	1    7100 1700
 	0    1    1    0
 $EndComp
@@
 L C C9
 U 1 1 58F2C556
-P 6850 2000
-F 0 "C9" V 6598 2000 50  0000 C CNN
-F 1 "33p" V 6689 2000 50  0000 C CNN
-F 2 "Capacitors_ThroughHole:C_Rect_L4.6mm_W2.0mm_P2.50mm_MKS02_FKP02" H 6888 1850 50  0001 C CNN
-F 3 "" H 6850 2000 50  0001 C CNN
-	1    6850 2000
+P 7100 2200
+F 0 "C9" V 6848 2200 50  0000 C CNN
+F 1 "33p" V 6939 2200 50  0000 C CNN
+F 2 "Capacitors_ThroughHole:C_Rect_L4.6mm_W2.0mm_P2.50mm_MKS02_FKP02" H 7138 2050 50  0001 C CNN
+F 3 "" H 7100 2200 50  0001 C CNN
+	1    7100 2200
 	0    1    1    0
 $EndComp
@@
 L GND #PWR019
 U 1 1 58F2C665
-P 6600 2150
-F 0 "#PWR019" H 6600 1900 50  0001 C CNN
-F 1 "GND" H 6605 1977 50  0000 C CNN
-F 2 "" H 6600 2150 50  0001 C CNN
-F 3 "" H 6600 2150 50  0001 C CNN
-	1    6600 2150
+P 6850 2350
+F 0 "#PWR019" H 6850 2100 50  0001 C CNN
+F 1 "GND" H 6855 2177 50  0000 C CNN
+F 2 "" H 6850 2350 50  0001 C CNN
+F 3 "" H 6850 2350 50  0001 C CNN
+	1    6850 2350
 	1    0    0    -1
 $EndComp
@@
 NoConn ~ 8300 3100
 NoConn ~ 8300 1100
-NoConn ~ 8900 250
-NoConn ~ 4350 250
 $Comp
 L Transformer_spitznagel_SPK01406 T1
@@
 Connection ~ 4300 1900
 Wire Wire Line
-	4300 1050 4300 1350
+	4300 600  4300 1350
 Connection ~ 4300 1050
 Wire Wire Line
@@
 	10550 1800 10850 1800
 Wire Wire Line
-	7000 1500 7450 1500
-Wire Wire Line
-	7100 1500 7100 1600
-Wire Wire Line
-	6700 1500 6600 1500
-Wire Wire Line
-	6600 1500 6600 2150
-Wire Wire Line
-	6700 2000 6600 2000
-Connection ~ 6600 2000
-Wire Wire Line
-	7000 2000 7450 2000
-Wire Wire Line
-	7100 2000 7100 1900
-Wire Wire Line
-	8300 1800 7450 1800
-Wire Wire Line
-	7450 1800 7450 2000
-Connection ~ 7100 2000
-Wire Wire Line
-	7450 1500 7450 1700
-Wire Wire Line
-	7450 1700 8300 1700
-Connection ~ 7100 1500
+	7250 1700 8300 1700
+Wire Wire Line
+	7350 1700 7350 1800
+Wire Wire Line
+	6950 1700 6850 1700
+Wire Wire Line
+	6850 1700 6850 2350
+Wire Wire Line
+	6950 2200 6850 2200
+Connection ~ 6850 2200
+Wire Wire Line
+	7250 2200 7700 2200
+Wire Wire Line
+	7350 2200 7350 2100
+Connection ~ 7350 2200
+Connection ~ 7350 1700
 Wire Notes Line
 	1900 800  1900 2450
@@
 F 0 "U1" H 4800 1417 50  0000 C CNN
 F 1 "LM7805CT" H 4800 1326 50  0000 C CNN
-F 2 "TO_SOT_Packages_THT:TO-220_Vertical" H 4800 1200 50  0001 C CIN
+F 2 "TO_SOT_Packages_THT:TO-220_Horizontal" H 4800 1200 50  0001 C CIN
 F 3 "" H 4800 1100 50  0001 C CNN
 	1    4800 1100
@@
 Connection ~ 3850 4000
 $Comp
-L iotta_logo CASE?
+L iotta_logo CASE1
 U 1 1 58F16C0B
 P 7150 6950
-F 0 "CASE?" H 7778 7103 60  0000 L CNN
+F 0 "CASE1" H 7778 7103 60  0000 L CNN
 F 1 "Case" H 7778 7050 60  0001 L CNN
 F 2 "iotta_footprints:CASE_KEMO_G085N" H 7778 6997 60  0000 L CNN
@@
 	1    0    0    -1
 $EndComp
+$Comp
+L AP111750 U6
+U 1 1 58F26D3E
+P 6700 800
+F 0 "U6" H 6700 1167 50  0000 C CNN
+F 1 "AP111750" H 6700 1076 50  0000 C CNN
+F 2 "TO_SOT_Packages_SMD:SOT-223" H 6700 450 50  0001 C CNN
+F 3 "" H 6800 550 50  0001 C CNN
+	1    6700 800
+	1    0    0    -1
+$EndComp
+Wire Wire Line
+	8300 1800 7700 1800
+Wire Wire Line
+	7700 1800 7700 2200
+$Comp
+L GND #PWR020
+U 1 1 58F2841B
+P 6700 1100
+F 0 "#PWR020" H 6700 850 50  0001 C CNN
+F 1 "GND" H 6705 927 50  0000 C CNN
+F 2 "" H 6700 1100 50  0001 C CNN
+F 3 "" H 6700 1100 50  0001 C CNN
+	1    6700 1100
+	1    0    0    -1
+$EndComp
+$Comp
+L VCC #PWR021
+U 1 1 58F2849C
+P 7100 750
+F 0 "#PWR021" H 7100 600 50  0001 C CNN
+F 1 "VCC" H 7117 923 50  0000 C CNN
+F 2 "" H 7100 750 50  0001 C CNN
+F 3 "" H 7100 750 50  0001 C CNN
+	1    7100 750
+	1    0    0    -1
+$EndComp
+Wire Wire Line
+	6400 800  6250 800
+Wire Wire Line
+	6250 800  6250 600
+Wire Wire Line
+	6250 600  4300 600
+Wire Wire Line
+	7000 800  7100 800
+Wire Wire Line
+	7100 800  7100 750
+Text Notes 7250 800  0    60   ~ 0
+1117 Regulator SMD alternative\nfor 7805 (place only one!)
+$Comp
+L iotta_logo WIRESTRAP1
+U 1 1 58F22411
+P 3400 7650
+F 0 "WIRESTRAP1" H 4028 7856 60  0000 L CNN
+F 1 "2x Ziplock wire strap" H 4028 7750 60  0000 L CNN
+F 2 "iotta_footprints:WireStrap_2X" H 4028 7644 60  0000 L CNN
+F 3 "" H 3400 7650 60  0000 C CNN
+	1    3400 7650
+	1    0    0    -1
+$EndComp
